Commit message: add to ros2_control velocity_controller

File: src/articubot_one/description/robot_core.xacro (robot description, xacro)
@@ -11,5 +11,5 @@
     <pose>0 0 0.1 0 0 0</pose>
     <inertial>
-      <mass value="15.0"/>
+      <mass value="150.0"/>
       <origin xyz="0.0 0 0" rpy=" 0 0 0"/>
       <inertia ixx="0.1" ixy="0" ixz="0" iyy="0.1" iyz="0" izz="0.1" />
@@ -148,5 +148,5 @@
     <parent link="chassis"/>
     <axis xyz="0 1 0" rpy="0 0 0"/>
-    <limit effort="10000" velocity="1000"/>
+    <limit effort="10" velocity="10"/>
     <dynamics damping="1.0" friction="1.0"/>
   </joint>
@@ -156,5 +156,5 @@
     <parent link="chassis"/>
     <axis xyz="0 1 0" rpy="0 0 0"/>
-    <limit effort="10000" velocity="1000"/>
+    <limit effort="10" velocity="10"/>
     <dynamics damping="1.0" friction="1.0"/>
   </joint>
@@ -164,5 +164,5 @@
     <parent link="chassis"/>
     <axis xyz="0 1 0" rpy="0 0 0"/>
-    <limit effort="10000" velocity="1000"/>
+    <limit effort="10" velocity="10"/>
     <dynamics damping="1.0" friction="1.0"/>
   </joint>
@@ -172,5 +172,5 @@
     <parent link="chassis"/>
     <axis xyz="0 1 0" rpy="0 0 0"/>
-    <limit effort="10000" velocity="1000"/>
+    <limit effort="10" velocity="10"/>
     <dynamics damping="1.0" friction="1.0"/>
   </joint>
