Commit message: diff_drive_controller add

File: src/articubot_one/description/ros2_control.xacro (robot description, xacro)
@@ -29,22 +29,4 @@
                 <state_interface name="effort" />
             </joint>
-            <joint name="lf_steering_hinge_joint">
-                <command_interface name="position">
-                    <param name="min">-0.5</param>
-                    <param name="max">0.5</param>
-                </command_interface>
-                <state_interface name="position" />
-                <state_interface name="velocity" />
-                <state_interface name="effort" />
-            </joint>
-            <joint name="rf_steering_hinge_joint">
-                <command_interface name="position">
-                    <param name="min">-0.5</param>
-                    <param name="max">0.5</param>
-                </command_interface>
-                <state_interface name="position" />
-                <state_interface name="velocity" />
-                <state_interface name="effort" />
-            </joint>
         </ros2_control>
     <gazebo>
